Commit message: .

File: URDF for Robot Modeling in ROS2/exemplos/marcos_bot_description/urdf/marcos_bot_simple.urdf (robot description, URDF)
Before this commit: robot urdfbot, 1 links, 0 joints
Links:
- added link head_link; visual box size=0.1 0.1 0.1
Joints:
- added joint base_link_to_head_link_joint: type revolute, parent base_link, child head_link, origin xyz=0 0 0.11 rpy=0 0 0, axis 0 0 1, limit lower=-1.57 upper=1.57 effort=100 velocity=1.0

Commit message: .

File: URDF for Robot Modeling in ROS2/exemplos/marcos_bot_description/urdf/marcos_bot_simple.urdf (robot description, URDF)
Before this commit: robot marcos_bot, 2 links, 1 joints
Links:
- link base_link: geometry visual mesh filename=package://marcos_bot_description/meshes/urdfbot_body.dae scale=0.1 0.1 0.1
- link head_link: geometry visual mesh filename=package://marcos_bot_description/meshes/urdfbot_head.dae scale=0.1 0.1 0.1
Joints:
- joint base_link_to_head_link_joint: origin xyz=0 0 0.11 rpy=0 0 0 -> xyz=0 0 0.07 rpy=0 0 0
