Commit message: .

File: URDF for Robot Modeling in ROS2/exemplos/marcos_box_bot_description/urdf/box_bot_geometric.urdf (robot description, URDF)
Before this commit: robot box_bot, 10 links, 9 joints
Links:
- link chassis: geometry collision box size=0.1 0.1 0.1; visual box size=0.1 0.1 0.1

File: URDF for Robot Modeling in ROS2/exemplos/marcos_box_bot_description/urdf/box_bot_geometric_meshes.urdf (robot description, URDF)
Before this commit: robot box_bot, 10 links, 9 joints
Links:
- link chassis: geometry collision mesh filename=package://marcos_box_bot_description/meshes/cute_cube.dae scale=0.1 0.1 0.1; visual mesh filename=package://marcos_box_bot_description/meshes/cute_cube.dae scale=0.1 0.1 0.1

Commit message: .

File: URDF for Robot Modeling in ROS2/exemplos/marcos_box_bot_description/urdf/box_bot_geometric.urdf (robot description, URDF)
Before this commit: robot box_bot, 10 links, 9 joints
Links:
- link back_roll_link: mass None -> 0.001; geometry collision cylinder length=0.001 radius=0.0045000000000000005; visual cylinder length=0.001 radius=0.0045
- link back_yaw_link: mass None -> 0.001; geometry collision cylinder length=0.001 radius=0.0045000000000000005; visual cylinder length=0.001 radius=0.0045
- link chassis: mass None -> 0.2
- link front_roll_link: mass None -> 0.001; geometry collision cylinder length=0.001 radius=0.0045000000000000005; visual cylinder length=0.001 radius=0.0045
- link front_yaw_link: mass None -> 0.001; geometry collision cylinder length=0.001 radius=0.0045000000000000005; visual cylinder length=0.001 radius=0.0045
- link left_wheel: mass None -> 0.05; geometry collision cylinder length=0.001 radius=0.035; visual cylinder length=0.001 radius=0.035

File: URDF for Robot Modeling in ROS2/exemplos/marcos_box_bot_description/urdf/box_bot_geometric_meshes.urdf (robot description, URDF)
Before this commit: robot box_bot, 10 links, 9 joints
Links:
- link chassis: mass None -> 0.2
